Commit message: Continuing work on xacro

File: mobilearmbot_description/urdf/mobilearmbot.urdf.xacro (robot description, xacro)
@@ -9,5 +9,27 @@
 	<xacro:property name="wheel_length" value="0.05"/>
 	<xacro:property name="wheel_mass" value="0.1"/>
-        <xacro:property name="pi" value="3.1415"/>
+	<xacro:property name="pi" value="3.1415"/>
+	<xacro:macro name="wheel_link_description">
+		<visual>
+			<origin rpy="${pi/2} 0 0" xyz="0 0 0"/>
+			<geometry>
+				<cylinder length="${wheel_length}" radius="${wheel_diam/2.0}"/>
+			</geometry>
+			<material name="black"/>
+		</visual>
+		<collision>
+			<origin rpy="${pi/2} 0 0" xyz="0 0 0"/>
+			<geometry>
+				<cylinder length="${wheel_length}" radius="${wheel_diam/2.0}"/>
+			</geometry>
+		</collision>
+		<inertial>
+			<mass value="${wheel_mass}"/>
+			<inertia ixx="${wheel_mass * (3*wheel_diam*wheel_diam/4.0 + wheel_length*wheel_length)/12.0}"
+				ixy="0.0" ixz="0.0"
+				iyy="${wheel_mass * (3*wheel_diam*wheel_diam/4.0 + wheel_length*wheel_length)/12.0}"
+				iyz="0.0" izz="${0.5*wheel_mass*wheel_diam*wheel_diam/4.0}"/>
+		</inertial>
+	</xacro:macro>
 	<!-- Base link -->
 	<link name="base_link">
@@ -35,21 +57,5 @@
 	<!-- Right front wheel -->
 	<link name="right_front_wheel">
-		<visual>
-			<origin rpy="1.57 0 0" xyz="0 0 0"/>
-			<geometry>
-				<cylinder length="0.05" radius="0.05"/>
-			</geometry>
-			<material name="black"/>
-		</visual>
-		<collision>
-			<origin rpy="1.57 0 0" xyz="0 0 0"/>
-			<geometry>
-				<cylinder length="0.05" radius="0.05"/>
-			</geometry>
-		</collision>
-		<inertial>
-			<mass value="0.1"/>
-			<inertia ixx="8.33e-05" ixy="0" ixz="0" iyy="8.33e-05" iyz="0" izz="1.25e-04"/>
-		</inertial>
+		<xacro:wheel_link_description />
 	</link>
 	<joint name="right_front_wheel_joint" type="continuous">
@@ -68,21 +74,5 @@
 	<!-- Right back wheel -->
 	<link name="right_back_wheel">
-		<visual>
-			<origin rpy="1.57 0 0" xyz="0 0 0"/>
-			<geometry>
-				<cylinder length="0.05" radius="0.05"/>
-			</geometry>
-			<material name="black"/>
-		</visual>
-		<collision>
-			<origin rpy="1.57 0 0" xyz="0 0 0"/>
-			<geometry>
-				<cylinder length="0.05" radius="0.05"/>
-			</geometry>
-		</collision>
-		<inertial>
-			<mass value="0.1"/>
-			<inertia ixx="8.33e-05" ixy="0" ixz="0" iyy="8.33e-05" iyz="0" izz="1.25e-04"/>
-		</inertial>
+		<xacro:wheel_link_description />
 	</link>
 	<joint name="right_back_wheel_joint" type="continuous">
@@ -101,21 +91,5 @@
 	<!-- Left front wheel -->
 	<link name="left_front_wheel">
-		<visual>
-			<origin rpy="1.57 0 0" xyz="0 0 0"/>
-			<geometry>
-				<cylinder length="0.05" radius="0.05"/>
-			</geometry>
-			<material name="black"/>
-		</visual>
-		<collision>
-			<origin rpy="1.57 0 0" xyz="0 0 0"/>
-			<geometry>
-				<cylinder length="0.05" radius="0.05"/>
-			</geometry>
-		</collision>
-		<inertial>
-			<mass value="0.1"/>
-			<inertia ixx="8.33e-05" ixy="0" ixz="0" iyy="8.33e-05" iyz="0" izz="1.25e-04"/>
-		</inertial>
+		<xacro:wheel_link_description />
 	</link>
 	<joint name="left_front_wheel_joint" type="continuous">
@@ -134,21 +108,5 @@
 	<!-- Left back wheel -->
 	<link name="left_back_wheel">
-		<visual>
-			<origin rpy="1.57 0 0" xyz="0 0 0"/>
-			<geometry>
-				<cylinder length="0.05" radius="0.05"/>
-			</geometry>
-			<material name="black"/>
-		</visual>
-		<collision>
-			<origin rpy="1.57 0 0" xyz="0 0 0"/>
-			<geometry>
-				<cylinder length="0.05" radius="0.05"/>
-			</geometry>
-		</collision>
-		<inertial>
-			<mass value="0.1"/>
-			<inertia ixx="8.33e-05" ixy="0" ixz="0" iyy="8.33e-05" iyz="0" izz="1.25e-04"/>
-		</inertial>
+		<xacro:wheel_link_description />
 	</link>
 	<joint name="left_back_wheel_joint" type="continuous">

Commit message: Used moveit assistant setup to create moveit package

File: mobilearmbot_description/urdf/mobilearmbot.urdf.xacro (robot description, xacro)
@@ -249,5 +249,5 @@
 		<child link="left_end_effector"/>
 		<origin rpy="0 0 0" xyz="0 ${link_radii} ${arm_link3_length}"/>
-		<axis xyz="0 1 0"/>
+		<axis xyz="1 0 0"/>
 	</joint>
 	<xacro:Transmission joint="left_end_effector_joint" n="3"/>
@@ -274,5 +274,5 @@
 		<child link="right_end_effector"/>
 		<origin rpy="0 0 0" xyz="0 ${-link_radii} ${arm_link3_length}"/>
-		<axis xyz="0 1 0"/>
+		<axis xyz="1 0 0"/>
 	</joint>
 	<xacro:Transmission joint="right_end_effector_joint" n="4"/>
