Commit message: Added collision and inertial details

File: mobilearmbot_description/urdf/mobilearmbot.urdf (robot description, URDF)
Before this commit: robot mobilearmbot, 5 links, 4 joints
Links:
- link base_link: mass None -> 3.0; geometry collision box size=0.3 0.3 0.15; visual box size=0.3 0.3 0.15
- link left_back_wheel: mass None -> 0.1; geometry collision cylinder length=0.05 radius=0.05; visual cylinder length=0.05 radius=0.05
- link left_front_wheel: mass None -> 0.1; geometry collision cylinder length=0.05 radius=0.05; visual cylinder length=0.05 radius=0.05
- link right_back_wheel: mass None -> 0.1; geometry collision cylinder length=0.05 radius=0.05; visual cylinder length=0.05 radius=0.05
- link right_front_wheel: mass None -> 0.1; geometry collision cylinder length=0.05 radius=0.05; visual cylinder length=0.05 radius=0.05

Commit message: Added laser scan

File: mobilearmbot_description/urdf/mobilearmbot.urdf (robot description, URDF)
Before this commit: robot mobilearmbot, 5 links, 4 joints
Links:
- added link laserscan, mass 0.01; collision box size=0.05 0.05 0.05; visual box size=0.05 0.05 0.05
Joints:
- added joint laserscan_joint: type fixed, parent base_link, child laserscan, origin xyz=0.1 0 0.10 rpy=0 0 0

Commit message: xacro and gazebo file caught up to urdf

File: mobilearmbot_description/urdf/mobilearmbot.urdf (robot description, URDF)
Before this commit: robot mobilearmbot, 6 links, 5 joints
Joints:
- joint left_back_wheel_joint: origin xyz=-0.075 0.155 -0.075 rpy=0 0 0 -> xyz=-0.05 0.155 -0.075 rpy=0 0 0
- joint left_front_wheel_joint: origin xyz=0.075 0.155 -0.075 rpy=0 0 0 -> xyz=0.05 0.155 -0.075 rpy=0 0 0
- joint right_back_wheel_joint: origin xyz=-0.075 -0.155 -0.075 rpy=0 0 0 -> xyz=-0.05 -0.155 -0.075 rpy=0 0 0
- joint right_front_wheel_joint: origin xyz=0.075 -0.155 -0.075 rpy=0 0 0 -> xyz=0.05 -0.155 -0.075 rpy=0 0 0

File: mobilearmbot_description/urdf/mobilearmbot.urdf.xacro (robot description, xacro)
@@ -2,8 +2,11 @@
 <robot name="mobilearmbot" xmlns:xacro="http://ros.org/wiki/xacro">
 	<xacro:include filename="$(find mobilearmbot_description)/urdf/colours.xacro"/>
+	<xacro:include filename="$(find mobilearmbot_description)/urdf/mobilearmbot.gazebo.xacro"/>
+	<!-- Constants for drivebase -->
 	<xacro:property name="base_length" value="0.3"/>
 	<xacro:property name="base_width" value="0.3"/>
 	<xacro:property name="base_height" value="0.15"/>
 	<xacro:property name="base_mass" value="3.0"/>
+	<!-- Constants & definition for the four wheels -->
 	<xacro:property name="wheel_diam" value="0.1"/>
 	<xacro:property name="wheel_length" value="0.05"/>
@@ -32,4 +35,9 @@
 		</inertial>
 	</xacro:macro>
+	<!-- Constants for laser scan-->
+	<xacro:property name="scan_length" value="0.05"/>
+	<xacro:property name="scan_width" value="0.05"/>
+	<xacro:property name="scan_height" value="0.05"/>
+	<xacro:property name="scan_mass" value="0.01"/>
 	<!-- Base link -->
 	<link name="base_link">
@@ -62,14 +70,7 @@
 		<parent link="base_link"/>
 		<child link="right_front_wheel"/>
-		<origin xyz="0.075 -0.155 -0.075" rpy="0 0 0"/>
+		<origin xyz="${base_length/4.0} ${-base_width/2.0 - 0.005} ${-base_height/2.0}" rpy="0 0 0"/>
 		<axis xyz="0 1 0"/>
 	</joint>
-	<gazebo reference="right_front_wheel">
-		<mu1 value="0.1"/>
-		<mu2 value="0.1"/>
-		<kp value="10000.0"/>
-		<kd value="1.0"/>
-		<material>Gazebo/Black</material>
-	</gazebo>
 	<!-- Right back wheel -->
 	<link name="right_back_wheel">
@@ -79,14 +80,7 @@
 		<parent link="base_link"/>
 		<child link="right_back_wheel"/>
-		<origin xyz="-0.075 -0.155 -0.075" rpy="0 0 0"/>
+		<origin xyz="${-base_length/4.0} ${-base_width/2.0 - 0.005} ${-base_height/2.0}" rpy="0 0 0"/>
 		<axis xyz="0 1 0"/>
 	</joint>
-        <gazebo reference="right_back_wheel">
-                <mu1 value="0.1"/>
-                <mu2 value="0.1"/>
-                <kp value="10000.0"/>
-                <kd value="1.0"/>
-                <material>Gazebo/Black</material>
-        </gazebo>
 	<!-- Left front wheel -->
 	<link name="left_front_wheel">
@@ -96,14 +90,7 @@
 		<parent link="base_link"/>
 		<child link="left_front_wheel"/>
-		<origin xyz="0.075 0.155 -0.075" rpy="0 0 0"/>
+		<origin xyz="${base_length/4.0} ${base_width/2.0 + 0.005} ${-base_height/2.0}" rpy="0 0 0"/>
 		<axis xyz="0 1 0"/>
 	</joint>
-        <gazebo reference="left_front_wheel">
-                <mu1 value="0.1"/>
-                <mu2 value="0.1"/>
-                <kp value="10000.0"/>
-                <kd value="1.0"/>
-                <material>Gazebo/Black</material>
-        </gazebo>
 	<!-- Left back wheel -->
 	<link name="left_back_wheel">
@@ -113,19 +100,12 @@
 		<parent link="base_link"/>
 		<child link="left_back_wheel"/>
-		<origin xyz="-0.075 0.155 -0.075" rpy="0 0 0"/>
+		<origin xyz="${-base_length/4.0} ${base_width/2.0 + 0.005} ${-base_height/2.0}" rpy="0 0 0"/>
 		<axis xyz="0 1 0"/>
 	</joint>
-        <gazebo reference="left_back_wheel">
-                <mu1 value="0.1"/>
-                <mu2 value="0.1"/>
-                <kp value="10000.0"/>
-                <kd value="1.0"/>
-                <material>Gazebo/Black</material>
-        </gazebo>
 	<link name="laserscan">
 		<visual>
 			<origin rpy="0 0 0" xyz="0 0 0"/>
 			<geometry>
-				<box size="0.05 0.05 0.05"/>
+				<box size="${scan_length} ${scan_width} ${scan_height}"/>
 			</geometry>
 			<material name="blue"/>
@@ -134,10 +114,13 @@
 			<origin rpy="0 0 0" xyz="0 0 0"/>
 			<geometry>
-				<box size="0.05 0.05 0.05"/>
+				<box size="${scan_length} ${scan_width} ${scan_height}"/>
 			</geometry>
 		</collision>
 		<inertial>
-			<mass value="0.01"/>
-			<inertia ixx="1.67e-7" iyy="1.67e-7" izz="1.67e-7" ixy="0" ixz="0" iyz="0"/>
+			<mass value="${scan_mass}"/>
+                        <inertia ixx="${scan_mass * (scan_height*scan_height + scan_length*scan_length)/12.0}"
+                                ixy="0.0" ixz="0.0"
+                                iyy="${scan_mass * (scan_width*scan_width + scan_length*scan_length)/12.0}"
+                                iyz="0.0" izz="${scan_mass * (scan_width*scan_width + scan_height*scan_height)/12.0}"/>
 		</inertial>
 	</link>
@@ -147,56 +130,3 @@
 		<origin xyz="0.1 0 0.10" rpy="0 0 0"/>
 	</joint>
-	<gazebo reference="laserscan">
-		<material>Gazebo/Black</material>
-		<sensor type="ray" name="laserscan1">
-			<pose>0 0 0 0 0 0</pose>
-			<visualize>false</visualize>
-			<update_rate>10</update_rate>
-			<ray>
-				<scan>
-					<horizontal>
-						<samples>360</samples>
-						<resolution>1</resolution>
-						<min_angle>0.0</min_angle>
-						<max_angle>6.28</max_angle>
-					</horizontal>
-				</scan>
-				<range>
-					<min>0.2</min>
-					<max>30.0</max>
-					<resolution>0.015</resolution>
-				</range>
-				<noise>
-					<type>gaussian</type>
-					<mean>0</mean>
-					<stddev>0.01</stddev>
-				</noise>
-			</ray>
-			<plugin name="mobilearmbot_laserscan_controller" filename="libgazebo_ros_laser.so">
-				<topicName>scan</topicName>
-				<frameName>base_scan</frameName>
-			</plugin>
-		</sensor>
-	</gazebo>
-	<gazebo>
-		<plugin name="mobilearmbot_controller" filename="libgazebo_ros_skid_steer_drive.so">
-			<updateRate>30.0</updateRate>
-			<robotNamespace>/</robotNamespace>
-			<leftFrontJoint>left_front_wheel_joint</leftFrontJoint>
-			<rightFrontJoint>right_front_wheel_joint</rightFrontJoint>
-			<leftRearJoint>left_back_wheel_joint</leftRearJoint>
-			<rightRearJoint>right_back_wheel_joint</rightRearJoint>
-			<wheelSeparation>0.3</wheelSeparation>
-			<wheelDiameter>0.1</wheelDiameter>
-			<robotBaseFrame>base_link</robotBaseFrame>
-			<torque>20</torque>
-			<topicName>cmd_vel</topicName>
-			<odometryTopic>odom</odometryTopic>
-			<odometryFrame>odom</odometryFrame>
-			<odometrySource>world</odometrySource>
-			<publishOdomTF>true</publishOdomTF>
-			<publishWheelJointState>true</publishWheelJointState>
-			<broadcastTF>true</broadcastTF>
-		</plugin>
-	</gazebo>
 </robot>

Commit message: Autogenerated urdf file

File: mobilearmbot_description/urdf/mobilearmbot.urdf (robot description, URDF)
Before this commit: robot mobilearmbot, 6 links, 5 joints
Links:
- link base_link: mass 5.0 -> 3.0
- link laserscan: mass 0.01 -> 0.1
Joints:
- joint left_back_wheel_joint: origin xyz=-0.05 0.155 -0.075 rpy=0 0 0 -> xyz=-0.1 0.17 -0.06 rpy=0 0 0
- joint left_front_wheel_joint: origin xyz=0.05 0.155 -0.075 rpy=0 0 0 -> xyz=0.1 0.17 -0.06 rpy=0 0 0
- joint right_back_wheel_joint: origin xyz=-0.05 -0.155 -0.075 rpy=0 0 0 -> xyz=-0.1 -0.17 -0.06 rpy=0 0 0
- joint right_front_wheel_joint: origin xyz=0.1 -0.175 -0.06 rpy=0 0 0 -> xyz=0.1 -0.17 -0.06 rpy=0 0 0

File: mobilearmbot_description/urdf/mobilearmbot.urdf.xacro (robot description, xacro)
@@ -42,4 +42,7 @@
 	<xacro:property name="scan_height" value="0.05"/>
 	<xacro:property name="scan_mass" value="0.1"/>
+	<!-- Constants for links -->
+	<xacro:property name="link1_length" value="0.5"/>
+	<xacro:property name="link1_radius" value="0.05"/>
 	<!-- Base link -->
 	<link name="base_link">

Commit message: moveit generated urdf is messed up

File: mobilearmbot_description/urdf/mobilearmbot.urdf (robot description, URDF)
Before this commit: robot mobilearmbot, 11 links, 10 joints
Links:
- link left_end_effector: mass None -> 0.1; geometry collision box size=0.1 0.05 0.01; visual box size=0.1 0.05 0.01
- link right_end_effector: mass None -> 0.1; geometry collision box size=0.1 0.05 0.01; visual box size=0.1 0.05 0.01
Joints:
- joint arm_link1_joint: origin xyz=0 0 0.075 rpy=0 0 0 -> xyz=-0.075 0 0.075 rpy=0 0 0
- joint left_end_effector_joint: axis 0 1 0 -> 1 0 0
- joint right_end_effector_joint: axis 0 1 0 -> 1 0 0

File: mobilearmbot_description/urdf/mobilearmbot.urdf.xacro (robot description, xacro)
@@ -48,12 +48,14 @@
 	<xacro:property name="arm_link3_length" value="0.2"/>
 	<xacro:property name="arm_link3_mass" value="0.8"/>
-	<xacro:macro name="Transmission" params="joint n">
-		<transmission name="tran${n}">
+	<!-- this is used wherever necessary for all joints -->
+	<xacro:macro name="Transmission" params="joint">
+		<transmission name="trans_${joint}">
 			<type>transmission_interface/SimpleTransmission</type>
 			<joint name="${joint}">
 				<hardwareInterface>hardware_interface/PositionJointInterface</hardwareInterface>
 			</joint>
-			<actuator name="motor${n}">
+			<actuator name="${joint}_motor">
 				<hardwareInterface>hardware_interface/PositionJointInterface</hardwareInterface>
+				<mechanicalReduction>1</mechanicalReduction>
 			</actuator>
 		</transmission>
@@ -95,4 +97,5 @@
 		<dynamics damping="${wheel_df}"/>
 	</joint>
+	<xacro:Transmission joint="right_front_wheel_joint"/>
 	<!-- Right back wheel -->
 	<link name="right_back_wheel">
@@ -106,4 +109,5 @@
 		<dynamics damping="${wheel_df}"/>
 	</joint>
+	<xacro:Transmission joint="right_back_wheel_joint"/>
 	<!-- Left front wheel -->
 	<link name="left_front_wheel">
@@ -117,4 +121,5 @@
 		<dynamics damping="${wheel_df}"/>
 	</joint>
+	<xacro:Transmission joint="left_front_wheel_joint"/>
 	<!-- Left back wheel -->
 	<link name="left_back_wheel">
@@ -128,4 +133,5 @@
 		<dynamics damping="${wheel_df}"/>
 	</joint>
+	<xacro:Transmission joint="left_back_wheel_joint"/>
 	<link name="base_scan">
 		<visual>
@@ -176,5 +182,5 @@
 		<axis xyz="0 0 1"/>
 	</joint>
-	<xacro:Transmission joint="arm_link1_joint" n="0"/>
+	<xacro:Transmission joint="arm_link1_joint"/>
 	<link name="arm_link2">
 		<visual>
@@ -201,5 +207,5 @@
 		<axis xyz="0 1 0"/>
 	</joint>
-	<xacro:Transmission joint="arm_link2_joint" n="1"/>
+	<xacro:Transmission joint="arm_link2_joint"/>
 	<link name="arm_link3">
 		<visual>
@@ -226,5 +232,5 @@
 		<axis xyz="0 1 0"/>
 	</joint>
-	<xacro:Transmission joint="arm_link3_joint" n="2"/>
+	<xacro:Transmission joint="arm_link3_joint"/>
 	<link name="left_end_effector">
 		<visual>
@@ -251,5 +257,5 @@
 		<axis xyz="1 0 0"/>
 	</joint>
-	<xacro:Transmission joint="left_end_effector_joint" n="3"/>
+	<xacro:Transmission joint="left_end_effector_joint"/>
 	<link name="right_end_effector">
 		<visual>
@@ -276,4 +282,4 @@
 		<axis xyz="1 0 0"/>
 	</joint>
-	<xacro:Transmission joint="right_end_effector_joint" n="4"/>
+	<xacro:Transmission joint="right_end_effector_joint"/>
 </robot>
