Commit message: Fixed tipping over issue

File: mobilearmbot_description/urdf/mobilearmbot.gazebo.xacro (robot description, xacro)
@@ -5,29 +5,13 @@
 	</gazebo>
 	<gazebo reference="right_front_wheel">
-		<mu1>0.1</mu1>
-		<mu2>0.1</mu2>
-		<kp>10000.0</kp>
-		<kd>10</kd>
 		<material>Gazebo/Black</material>
 	</gazebo>
         <gazebo reference="right_back_wheel">
-                <mu1>0.1</mu1>
-                <mu2>0.1</mu2>
-                <kp>10000.0</kp>
-                <kd>10</kd>
                 <material>Gazebo/Black</material>
 	</gazebo>
         <gazebo reference="left_front_wheel">
-                <mu1>0.1</mu1>
-                <mu2>0.1</mu2>
-                <kp>10000.0</kp>
-                <kd>10</kd>
                 <material>Gazebo/Black</material>
 	</gazebo>
         <gazebo reference="left_back_wheel">
-                <mu1>0.1</mu1>
-                <mu2>0.1</mu2>
-                <kp>10000.0</kp>
-                <kd>10</kd>
                 <material>Gazebo/Black</material>
 	</gazebo>
@@ -72,5 +56,5 @@
                         <leftRearJoint>left_back_wheel_joint</leftRearJoint>
                         <rightRearJoint>right_back_wheel_joint</rightRearJoint>
-                        <wheelSeparation>0.3</wheelSeparation>
+                        <wheelSeparation>0.67</wheelSeparation>
                         <wheelDiameter>0.1</wheelDiameter>
                         <robotBaseFrame>base_link</robotBaseFrame>

File: mobilearmbot_description/urdf/mobilearmbot.urdf (robot description, URDF)
Before this commit: robot mobilearmbot, 6 links, 5 joints
Links:
- link base_link: mass 3.0 -> 5.0
- link left_back_wheel: mass 0.1 -> 1
- link left_front_wheel: mass 0.1 -> 1
- link right_back_wheel: mass 0.1 -> 1
- link right_front_wheel: mass 0.1 -> 1
Joints:
- joint right_front_wheel_joint: origin xyz=0.05 -0.155 -0.075 rpy=0 0 0 -> xyz=0.1 -0.175 -0.06 rpy=0 0 0

File: mobilearmbot_description/urdf/mobilearmbot.urdf.xacro (robot description, xacro)
@@ -11,6 +11,8 @@
 	<xacro:property name="wheel_diam" value="0.1"/>
 	<xacro:property name="wheel_length" value="0.05"/>
-	<xacro:property name="wheel_mass" value="0.1"/>
+	<xacro:property name="wheel_mass" value="1"/>
+	<xacro:property name="wheel_base_offset" value="0.02"/>
 	<xacro:property name="pi" value="3.1415"/>
+	<xacro:property name="wheel_df" value="0.0"/>
 	<xacro:macro name="wheel_link_description">
 		<visual>
@@ -39,5 +41,5 @@
 	<xacro:property name="scan_width" value="0.05"/>
 	<xacro:property name="scan_height" value="0.05"/>
-	<xacro:property name="scan_mass" value="0.01"/>
+	<xacro:property name="scan_mass" value="0.1"/>
 	<!-- Base link -->
 	<link name="base_link">
@@ -57,4 +59,5 @@
 		<inertial>
 			<mass value="${base_mass}"/>
+			<inertia ixx="1.0" ixy="0.0" ixz="0.0" iyy="1.0" iyz="0.0" izz="1.0"/>
 			<inertia ixx="${base_mass * (base_height*base_height + base_length*base_length)/12.0}"
 				ixy="0.0" ixz="0.0"
@@ -70,6 +73,7 @@
 		<parent link="base_link"/>
 		<child link="right_front_wheel"/>
-		<origin xyz="${base_length/4.0} ${-base_width/2.0 - 0.005} ${-base_height/2.0}" rpy="0 0 0"/>
+		<origin xyz="${base_length/3.0} ${-base_width/2.0 - wheel_base_offset} ${-base_height/2.5}" rpy="0 0 0"/>
 		<axis xyz="0 1 0"/>
+		<dynamics damping="${wheel_df}"/>
 	</joint>
 	<!-- Right back wheel -->
@@ -80,6 +84,7 @@
 		<parent link="base_link"/>
 		<child link="right_back_wheel"/>
-		<origin xyz="${-base_length/4.0} ${-base_width/2.0 - 0.005} ${-base_height/2.0}" rpy="0 0 0"/>
+		<origin xyz="${-base_length/3.0} ${-base_width/2.0 - wheel_base_offset} ${-base_height/2.5}" rpy="0 0 0"/>
 		<axis xyz="0 1 0"/>
+		<dynamics damping="${wheel_df}"/>
 	</joint>
 	<!-- Left front wheel -->
@@ -90,6 +95,7 @@
 		<parent link="base_link"/>
 		<child link="left_front_wheel"/>
-		<origin xyz="${base_length/4.0} ${base_width/2.0 + 0.005} ${-base_height/2.0}" rpy="0 0 0"/>
+		<origin xyz="${base_length/3.0} ${base_width/2.0 + wheel_base_offset} ${-base_height/2.5}" rpy="0 0 0"/>
 		<axis xyz="0 1 0"/>
+		<dynamics damping="${wheel_df}"/>
 	</joint>
 	<!-- Left back wheel -->
@@ -100,6 +106,7 @@
 		<parent link="base_link"/>
 		<child link="left_back_wheel"/>
-		<origin xyz="${-base_length/4.0} ${base_width/2.0 + 0.005} ${-base_height/2.0}" rpy="0 0 0"/>
+		<origin xyz="${-base_length/3.0} ${base_width/2.0 + wheel_base_offset} ${-base_height/2.5}" rpy="0 0 0"/>
 		<axis xyz="0 1 0"/>
+		<dynamics damping="${wheel_df}"/>
 	</joint>
 	<link name="laserscan">

Commit message: Cleaning up xacro further

File: mobilearmbot_description/urdf/mobilearmbot.gazebo.xacro (robot description, xacro)
@@ -16,7 +16,7 @@
                 <material>Gazebo/Black</material>
 	</gazebo>
-	<gazebo reference="laserscan">
+	<gazebo reference="base_scan">
                 <material>Gazebo/Black</material>
-                <sensor type="ray" name="laserscan1">
+                <sensor type="ray" name="laserscan">
                         <pose>0 0 0 0 0 0</pose>
                         <visualize>false</visualize>

File: mobilearmbot_description/urdf/mobilearmbot.urdf (robot description, URDF)
Before this commit: robot mobilearmbot, 6 links, 5 joints
Links:
- removed link laserscan
- added link arm_link1, mass 0.1; collision cylinder length=0.3 radius=0.05; visual cylinder length=0.3 radius=0.05
- added link arm_link2; visual cylinder length=0.4 radius=0.05
- added link base_scan, mass 0.1; collision box size=0.05 0.05 0.05; visual box size=0.05 0.05 0.05
Joints:
- removed joint laserscan_joint
- added joint arm_link1_joint: type continuous, parent base_link, child arm_link1, origin xyz=0 0 0.075 rpy=0 0 0, axis 0 0 1
- added joint arm_link2_joint: type continuous, parent arm_link1, child arm_link2, origin xyz=0 -0.1 0.3 rpy=0 1.57 0, axis 0 1 0
- added joint base_scan_joint: type fixed, parent base_link, child base_scan, origin xyz=0.1 0 0.1 rpy=0 0 0

File: mobilearmbot_description/urdf/mobilearmbot.urdf.xacro (robot description, xacro)
@@ -3,4 +3,5 @@
 	<xacro:include filename="$(find mobilearmbot_description)/urdf/colours.xacro"/>
 	<xacro:include filename="$(find mobilearmbot_description)/urdf/mobilearmbot.gazebo.xacro"/>
+	<xacro:include filename="$(find mobilearmbot_description)/urdf/inertias.xacro"/>
 	<!-- Constants for drivebase -->
 	<xacro:property name="base_length" value="0.3"/>
@@ -31,8 +32,5 @@
 		<inertial>
 			<mass value="${wheel_mass}"/>
-			<inertia ixx="${wheel_mass * (3*wheel_diam*wheel_diam/4.0 + wheel_length*wheel_length)/12.0}"
-				ixy="0.0" ixz="0.0"
-				iyy="${wheel_mass * (3*wheel_diam*wheel_diam/4.0 + wheel_length*wheel_length)/12.0}"
-				iyz="0.0" izz="${0.5*wheel_mass*wheel_diam*wheel_diam/4.0}"/>
+			<xacro:cylinder_inertia mass="${wheel_mass}" length="${wheel_length}" radius="${wheel_diam/2.0}"/>
 		</inertial>
 	</xacro:macro>
@@ -43,6 +41,9 @@
 	<xacro:property name="scan_mass" value="0.1"/>
 	<!-- Constants for links -->
-	<xacro:property name="link1_length" value="0.5"/>
-	<xacro:property name="link1_radius" value="0.05"/>
+	<xacro:property name="link_radii" value="0.05"/> <!-- All links will have the same radius -->
+	<xacro:property name="arm_link1_length" value="0.3"/>
+	<xacro:property name="arm_link2_length" value="0.4"/>
+	<xacro:property name="arm_link1_mass" value="1.2"/>
+	<xacro:property name="arm_link2_mass" value="1.6"/>
 	<!-- Base link -->
 	<link name="base_link">
@@ -62,9 +63,5 @@
 		<inertial>
 			<mass value="${base_mass}"/>
-			<inertia ixx="1.0" ixy="0.0" ixz="0.0" iyy="1.0" iyz="0.0" izz="1.0"/>
-			<inertia ixx="${base_mass * (base_height*base_height + base_length*base_length)/12.0}"
-				ixy="0.0" ixz="0.0"
-				iyy="${base_mass * (base_width*base_width + base_length*base_length)/12.0}"
-				iyz="0.0" izz="${base_mass * (base_width*base_width + base_height*base_height)/12.0}"/>
+			<xacro:box_inertia mass="${base_mass}" length="${base_length}" width="${base_width}" height="${base_height}"/>
 		</inertial>
 	</link>
@@ -113,5 +110,5 @@
 		<dynamics damping="${wheel_df}"/>
 	</joint>
-	<link name="laserscan">
+	<link name="base_scan">
 		<visual>
 			<origin rpy="0 0 0" xyz="0 0 0"/>
@@ -129,13 +126,10 @@
 		<inertial>
 			<mass value="${scan_mass}"/>
-                        <inertia ixx="${scan_mass * (scan_height*scan_height + scan_length*scan_length)/12.0}"
-                                ixy="0.0" ixz="0.0"
-                                iyy="${scan_mass * (scan_width*scan_width + scan_length*scan_length)/12.0}"
-                                iyz="0.0" izz="${scan_mass * (scan_width*scan_width + scan_height*scan_height)/12.0}"/>
+			<xacro:box_inertia mass="${scan_mass}" length="${scan_length}" width="${scan_width}" height="${scan_height}"/>
 		</inertial>
 	</link>
-	<joint name="laserscan_joint" type="fixed">
+	<joint name="base_scan_joint" type="fixed">
 		<parent link="base_link"/>
-		<child link="laserscan"/>
+		<child link="base_scan"/>
 		<origin xyz="0.1 0 0.10" rpy="0 0 0"/>
 	</joint>

Commit message: Added badly made arms

File: mobilearmbot_description/urdf/mobilearmbot.gazebo.xacro (robot description, xacro)
@@ -69,3 +69,8 @@
                 </plugin>
 	</gazebo>
+	<gazebo>
+		<plugin name="gazebo_ros_control" filename="libgazebo_ros_control.so">
+			<robotNamespace>/</robotNamespace>
+		</plugin>
+	</gazebo>
 </robot>

File: mobilearmbot_description/urdf/mobilearmbot.urdf (robot description, URDF)
Before this commit: robot mobilearmbot, 8 links, 7 joints
Links:
- link arm_link1: mass 0.1 -> 1.2
- link arm_link2: mass None -> 1.6; geometry collision cylinder length=0.4 radius=0.05; visual cylinder length=0.4 radius=0.05
Joints:
- joint arm_link2_joint: origin xyz=0 -0.1 0.3 rpy=0 1.57 0 -> xyz=0 0 0.3 rpy=0 1.57075 0

File: mobilearmbot_description/urdf/mobilearmbot.urdf.xacro (robot description, xacro)
@@ -46,4 +46,15 @@
 	<xacro:property name="arm_link1_mass" value="1.2"/>
 	<xacro:property name="arm_link2_mass" value="1.6"/>
+	<xacro:macro name="Transmission" params="joint n">
+		<transmission name="tran${n}">
+			<type>transmission_interface/SimpleTransmission</type>
+			<joint name="${joint}">
+				<hardwareInterface>hardware_interface/PositionJointInterface</hardwareInterface>
+			</joint>
+			<actuator name="motor${n}">
+				<hardwareInterface>hardware_interface/PositionJointInterface</hardwareInterface>
+			</actuator>
+		</transmission>
+	</xacro:macro>
 	<!-- Base link -->
 	<link name="base_link">
@@ -132,5 +143,55 @@
 		<parent link="base_link"/>
 		<child link="base_scan"/>
-		<origin xyz="0.1 0 0.10" rpy="0 0 0"/>
+		<origin xyz="0.1 0 ${scan_height/2.0 + base_height/2.0}" rpy="0 0 0"/>
 	</joint>
+	<link name="arm_link1">
+		<visual>
+			<origin rpy="0 0 0" xyz="0 0 ${arm_link1_length/2.0}"/>
+			<geometry>
+				<cylinder length="${arm_link1_length}" radius="${link_radii}"/>
+			</geometry>
+		</visual>
+		<collision>
+			<origin rpy="0 0 0" xyz="0 0 ${arm_link1_length/2.0}"/>
+			<geometry>
+				<cylinder length="${arm_link1_length}" radius="${link_radii}"/>
+			</geometry>
+		</collision>
+		<inertial>
+			<mass value="${arm_link1_mass}"/>
+			<xacro:cylinder_inertia mass="${arm_link1_mass}" length="${arm_link1_length}" radius="${link_radii}"/>
+		</inertial>
+	</link>
+	<joint name="arm_link1_joint" type="continuous">
+		<parent link="base_link"/>
+		<child link="arm_link1"/>
+		<origin rpy="0 0 0" xyz="0 0 ${base_height/2.0}"/>
+		<axis xyz="0 0 1"/>
+	</joint>
+	<xacro:Transmission joint="arm_link1_joint" n="0"/>
+	<link name="arm_link2">
+		<visual>
+			<origin rpy="0 0 0" xyz="0 0 ${arm_link2_length/2.0}"/>
+			<geometry>
+				<cylinder length="${arm_link2_length}" radius="${link_radii}"/>
+			</geometry>
+		</visual>
+		<collision>
+			<origin rpy="0 0 0" xyz="0 0 ${arm_link2_length/2.0}"/>
+			<geometry>
+				<cylinder length="${arm_link2_length}" radius="${link_radii}"/>
+			</geometry>
+		</collision>
+		<inertial>
+			<mass value="${arm_link2_mass}"/>
+			<xacro:cylinder_inertia mass="${arm_link2_mass}" length="${arm_link2_length}" radius="${link_radii}"/>
+		</inertial>
+	</link>
+	<joint name="arm_link2_joint" type="continuous">
+		<parent link="arm_link1"/>
+		<child link="arm_link2"/>
+		<origin rpy="0 ${pi/2} 0" xyz="0 0 ${arm_link1_length}"/>
+		<axis xyz="0 1 0"/>
+	</joint>
+	<xacro:Transmission joint="arm_link2_joint" n="1"/>
 </robot>

Commit message: Added another joint & end effector

File: mobilearmbot_description/urdf/mobilearmbot.gazebo.xacro (robot description, xacro)
@@ -15,4 +15,19 @@
         <gazebo reference="left_back_wheel">
                 <material>Gazebo/Black</material>
+	</gazebo>
+	<gazebo reference="arm_link1">
+		<material>Gazebo/Black</material>
+	</gazebo>
+	<gazebo reference="arm_link2">
+		<material>Gazebo/Black</material>
+	</gazebo>
+	<gazebo reference="arm_link3">
+		<material>Gazebo/Black</material>
+	</gazebo>
+	<gazebo reference="left_end_effector">
+		<material>Gazebo/Grey</material>
+	</gazebo>
+	<gazebo reference="right_end_effector">
+		<material>Gazebo/Grey</material>
 	</gazebo>
 	<gazebo reference="base_scan">

File: mobilearmbot_description/urdf/mobilearmbot.urdf (robot description, URDF)
Before this commit: robot mobilearmbot, 8 links, 7 joints
Links:
- added link arm_link3, mass 0.8; collision cylinder length=0.2 radius=0.05; visual cylinder length=0.2 radius=0.05
- added link left_end_effector; visual box size=0.1 0.05 0.01
- added link right_end_effector; visual box size=0.1 0.05 0.01
Joints:
- added joint arm_link3_joint: type continuous, parent arm_link2, child arm_link3, origin xyz=0 0 0.4 rpy=0 1.57075 0, axis 0 1 0
- added joint left_end_effector_joint: type continuous, parent arm_link3, child left_end_effector, origin xyz=0 0.05 0.2 rpy=0 0 0, axis 0 1 0
- added joint right_end_effector_joint: type continuous, parent arm_link3, child right_end_effector, origin xyz=0 -0.05 0.2 rpy=0 0 0, axis 0 1 0

File: mobilearmbot_description/urdf/mobilearmbot.urdf.xacro (robot description, xacro)
@@ -40,5 +40,5 @@
 	<xacro:property name="scan_height" value="0.05"/>
 	<xacro:property name="scan_mass" value="0.1"/>
-	<!-- Constants for links -->
+	<!-- Constants for arm links -->
 	<xacro:property name="link_radii" value="0.05"/> <!-- All links will have the same radius -->
 	<xacro:property name="arm_link1_length" value="0.3"/>
@@ -46,4 +46,6 @@
 	<xacro:property name="arm_link1_mass" value="1.2"/>
 	<xacro:property name="arm_link2_mass" value="1.6"/>
+	<xacro:property name="arm_link3_length" value="0.2"/>
+	<xacro:property name="arm_link3_mass" value="0.8"/>
 	<xacro:macro name="Transmission" params="joint n">
 		<transmission name="tran${n}">
@@ -57,4 +59,9 @@
 		</transmission>
 	</xacro:macro>
+	<!-- Constants for end effector -->
+	<xacro:property name="end_effector_length" value="0.1"/>
+	<xacro:property name="end_effector_width" value="0.05"/>
+	<xacro:property name="end_effector_height" value="0.01"/>
+	<xacro:property name="end_effector_mass" value="0.1"/>
 	<!-- Base link -->
 	<link name="base_link">
@@ -166,5 +173,5 @@
 		<parent link="base_link"/>
 		<child link="arm_link1"/>
-		<origin rpy="0 0 0" xyz="0 0 ${base_height/2.0}"/>
+		<origin rpy="0 0 0" xyz="${-base_height/2.0} 0 ${base_height/2.0}"/>
 		<axis xyz="0 0 1"/>
 	</joint>
@@ -195,3 +202,78 @@
 	</joint>
 	<xacro:Transmission joint="arm_link2_joint" n="1"/>
+	<link name="arm_link3">
+		<visual>
+			<origin rpy="0 0 0" xyz="0 0 ${arm_link3_length/2.0}"/>
+			<geometry>
+				<cylinder length="${arm_link3_length}" radius="${link_radii}"/>
+			</geometry>
+		</visual>
+		<collision>
+			<origin rpy="0 0 0" xyz="0 0 ${arm_link3_length/2.0}"/>
+			<geometry>
+				<cylinder length="${arm_link3_length}" radius="${link_radii}"/>
+			</geometry>
+		</collision>
+		<inertial>
+			<mass value="${arm_link3_mass}"/>
+			<xacro:cylinder_inertia mass="${arm_link3_mass}" length="${arm_link3_length}" radius="${link_radii}"/>
+		</inertial>
+	</link>
+	<joint name="arm_link3_joint" type="continuous">
+		<parent link="arm_link2"/>
+		<child link="arm_link3"/>
+		<origin rpy="0 ${pi/2} 0" xyz="0 0 ${arm_link2_length}"/>
+		<axis xyz="0 1 0"/>
+	</joint>
+	<xacro:Transmission joint="arm_link3_joint" n="2"/>
+	<link name="left_end_effector">
+		<visual>
+			<origin rpy="${pi/2} ${pi/2} 0" xyz="0 0 ${end_effector_length/2}"/>
+			<geometry>
+				<box size="${end_effector_length} ${end_effector_width} ${end_effector_height}"/>
+			</geometry>
+		</visual>
+		<collision>
+			<origin rpy="${pi/2} ${pi/2} 0" xyz="0 0 ${end_effector_length/2}"/>
+			<geometry>
+				<box size="${end_effector_length} ${end_effector_width} ${end_effector_height}"/>
+			</geometry>
+		</collision>
+		<inertial>
+			<mass value="${end_effector_mass}"/>
+			<xacro:box_inertia mass="${end_effector_mass}" length="${end_effector_length}" width="${end_effector_width}" height="${end_effector_height}"/>
+		</inertial>
+	</link>
+	<joint name="left_end_effector_joint" type="continuous">
+		<parent link="arm_link3"/>
+		<child link="left_end_effector"/>
+		<origin rpy="0 0 0" xyz="0 ${link_radii} ${arm_link3_length}"/>
+		<axis xyz="0 1 0"/>
+	</joint>
+	<xacro:Transmission joint="left_end_effector_joint" n="3"/>
+	<link name="right_end_effector">
+		<visual>
+			<origin rpy="${pi/2} ${pi/2} 0" xyz="0 0 ${end_effector_length/2}"/>
+			<geometry>
+				<box size="${end_effector_length} ${end_effector_width} ${end_effector_height}"/>
+			</geometry>
+		</visual>
+		<collision>
+                        <origin rpy="${pi/2} ${pi/2} 0" xyz="0 0 ${end_effector_length/2}"/>
+                        <geometry>
+                                <box size="${end_effector_length} ${end_effector_width} ${end_effector_height}"/>
+                        </geometry>
+		</collision>
+                <inertial>
+                        <mass value="${end_effector_mass}"/>
+                        <xacro:box_inertia mass="${end_effector_mass}" length="${end_effector_length}" width="${end_effector_width}" height="${end_effector_height}"/>
+                </inertial>
+	</link>
+	<joint name="right_end_effector_joint" type="continuous">
+		<parent link="arm_link3"/>
+		<child link="right_end_effector"/>
+		<origin rpy="0 0 0" xyz="0 ${-link_radii} ${arm_link3_length}"/>
+		<axis xyz="0 1 0"/>
+	</joint>
+	<xacro:Transmission joint="right_end_effector_joint" n="4"/>
 </robot>

Commit message: Fixed controller for drivetrain & moved starting config of end effector

File: mobilearmbot_description/urdf/mobilearmbot.gazebo.xacro (robot description, xacro)
@@ -47,5 +47,5 @@
                                 </scan>
                                 <range>
-                                        <min>0.2</min>
+                                        <min>0.3</min>
                                         <max>30.0</max>
                                         <resolution>0.015</resolution>

File: mobilearmbot_description/urdf/mobilearmbot.urdf (robot description, URDF)
Before this commit: robot mobilearmbot, 11 links, 10 joints
Joints:
- joint base_scan_joint: origin xyz=0.1 0 0.1 rpy=0 0 0 -> xyz=0.0 0 0.1 rpy=0 0 0
- joint left_end_effector_joint: origin xyz=0 0.05 0.2 rpy=0 0 0 -> xyz=0 0.05 0.2 rpy=-1.57075 0 0
- joint right_end_effector_joint: origin xyz=0 -0.05 0.2 rpy=0 0 0 -> xyz=0 -0.05 0.2 rpy=1.57075 0 0

File: mobilearmbot_description/urdf/mobilearmbot.urdf.xacro (robot description, xacro)
@@ -156,5 +156,5 @@
 		<parent link="base_link"/>
 		<child link="base_scan"/>
-		<origin xyz="0.1 0 ${scan_height/2.0 + base_height/2.0}" rpy="0 0 0"/>
+		<origin xyz="0.0 0 ${scan_height/2.0 + base_height/2.0}" rpy="0 0 0"/>
 	</joint>
 	<link name="arm_link1">
@@ -254,5 +254,5 @@
 		<parent link="arm_link3"/>
 		<child link="left_end_effector"/>
-		<origin rpy="0 0 0" xyz="0 ${link_radii} ${arm_link3_length}"/>
+		<origin rpy="${-pi/2} 0 0" xyz="0 ${link_radii} ${arm_link3_length}"/>
 		<axis xyz="1 0 0"/>
 	</joint>
@@ -279,5 +279,5 @@
 		<parent link="arm_link3"/>
 		<child link="right_end_effector"/>
-		<origin rpy="0 0 0" xyz="0 ${-link_radii} ${arm_link3_length}"/>
+		<origin rpy="${pi/2} 0 0" xyz="0 ${-link_radii} ${arm_link3_length}"/>
 		<axis xyz="1 0 0"/>
 	</joint>

Commit message: Currently have a typo somewhere

File: mobilearmbot_description/urdf/mobilearmbot.gazebo.xacro (robot description, xacro)
@@ -86,5 +86,5 @@
 	<gazebo>
 		<plugin name="gazebo_ros_control" filename="libgazebo_ros_control.so">
-			<robotNamespace>/</robotNamespace>
+			<robotNamespace>/mobilearmbot</robotNamespace>
 		</plugin>
 	</gazebo>

File: mobilearmbot_description/urdf/mobilearmbot.urdf.xacro (robot description, xacro)
@@ -66,4 +66,7 @@
 	<xacro:property name="end_effector_height" value="0.01"/>
 	<xacro:property name="end_effector_mass" value="0.1"/>
+	<!-- Fixed link -->
+	<link name="odom">
+	</link>
 	<!-- Base link -->
 	<link name="base_link">
@@ -86,4 +89,8 @@
 		</inertial>
 	</link>
+	<joint name="odom_joint" type="fixed">
+		<parent link="odom"/>
+		<child link="base_link"/>
+	</joint>
 	<!-- Right front wheel -->
 	<link name="right_front_wheel">

Commit message: Moveit working via rviz

File: mobilearmbot_description/urdf/mobilearmbot.gazebo.xacro (robot description, xacro)
@@ -59,5 +59,5 @@
 			<plugin name="mobilearmbot_laserscan_controller" filename="libgazebo_ros_laser.so">
 				<robotNamespace>/mobilearmbot</robotNamespace>
-                                <topicName>scan</topicName>
+				<topicName>scan</topicName>
                                 <frameName>base_scan</frameName>
                         </plugin>
@@ -66,6 +66,6 @@
         <gazebo>
                 <plugin name="mobilearmbot_controller" filename="libgazebo_ros_skid_steer_drive.so">
-                        <updateRate>30.0</updateRate>
-                        <robotNamespace>/mobilearmbot</robotNamespace>
+			<updateRate>30.0</updateRate>
+			<robotNamespace>/mobilearmbot</robotNamespace>
                         <leftFrontJoint>left_front_wheel_joint</leftFrontJoint>
                         <rightFrontJoint>right_front_wheel_joint</rightFrontJoint>

File: mobilearmbot_description/urdf/mobilearmbot.urdf (robot description, URDF)
Before this commit: robot mobilearmbot, 12 links, 11 joints
Links:
- removed link dummy
- added link odom
Joints:
- removed joint dummy_joint
- added joint odom_joint: type fixed, parent odom, child base_link
